Commit message: model color added

File: autonomousPro/src/robot_description/urdf/Assembly-Robot-URDF.urdf.xacro (robot description, xacro)
@@ -537,4 +537,5 @@
     <minDepth>0.001</minDepth>
     <maxVel>1.0</maxVel>
+    <material>Gazebo/Black</material>
   </gazebo>
   <gazebo reference="right_wheel_link">
@@ -546,4 +547,5 @@
     <minDepth>0.001</minDepth>
     <maxVel>1.0</maxVel>
+    <material>Gazebo/Black</material>
   </gazebo>
   <gazebo reference="front_wheel_link">
@@ -555,4 +557,5 @@
     <minDepth>0.001</minDepth>
     <maxVel>1.0</maxVel>
+    <material>Gazebo/Black</material>
   </gazebo>
   <gazebo reference="rear_wheel_link">
@@ -564,4 +567,5 @@
     <minDepth>0.001</minDepth>
     <maxVel>1.0</maxVel>
+    <material>Gazebo/Black</material>
   </gazebo>
 </robot>

File: autonomousPro/src/robot_description/urdf/common_properties.xacro (robot description, xacro)
@@ -45,3 +45,27 @@
     </inertial>
   </xacro:macro>
+    <gazebo reference="base_link">
+    <material>Gazebo/Grey</material>
+    </gazebo>
+    <gazebo reference="front_hinge">
+    <material>Gazebo/Grey</material>
+    </gazebo>
+    <gazebo reference="front_wheel_link">
+    <material>Gazebo/Black</material>
+    </gazebo>
+    <gazebo reference="left_wheel_link">
+    <material>Gazebo/Black</material>
+    </gazebo>
+    <gazebo reference="rear_hinge">
+    <material>Gazebo/Grey</material>
+    </gazebo>
+    <gazebo reference="rear_wheel_link">
+    <material>Gazebo/Black</material>
+    </gazebo>
+    <gazebo reference="right_wheel_link">
+    <material>Gazebo/Black</material>
+    </gazebo>
+    <gazebo reference="lidar_link">
+    <material>Gazebo/Blue</material>
+    </gazebo>
 </robot>
